File: driver_v0.2/driver.kicad_pcb (KiCad board)
At the start: 2 copper layers, 100 x 35 mm, 52 parts, among them J1 Pwr, J2 Batt, J3 isp, J4 Conn_02x05_Odd_Even, J5 Conn_01x06, J6 Conn_01x06, K1 Brake, Q1 IRF540N, Q2 NPN, Q3 NPN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

Commit message: 2021-09-04
Parts:
- removed K1: Brake, OPL_Switch:SW4-6.0X6.0X5.0MM
- removed R27: 10k, Resistor_SMD:R_0603_1608Metric_Pad0.98x0.95mm_HandSolder
- removed U3: MCP6044T-I_ST, MCP6044T:MCP6044T
- added Q10: BC846, Package_TO_SOT_SMD:SOT-23, F.Cu at (33.0, 9.00)
- added Q11: BC846, Package_TO_SOT_SMD:SOT-23, F.Cu at (17.5, 7.00)
- added Q8: BC856B, Package_TO_SOT_SMD:SOT-23, F.Cu at (22.0, 7.00)
- added Q9: NPN, Package_TO_SOT_SMD:SOT-23, F.Cu at (33.0, 4.00)
- added SW1: SW_Push, Button_Switch_THT:SW_PUSH_6mm, F.Cu at (7.00, 26.0)
- J3: value isp -> Conn_01x04; footprint Connector_JST:JST_PH_B6B-PH-K_1x06_P2.00mm_Vertical -> Connector_PinHeader_2.54mm:PinHeader_1x04_P2.54mm_Vertical
- J4: value Conn_02x05_Odd_Even -> Conn_01x06; footprint Connector_PinHeader_2.54mm:PinHeader_2x05_P2.54mm_Vertical -> Connector_JST:JST_PH_B6B-PH-K_1x06_P2.00mm_Vertical
- J6: value Conn_01x06 -> Conn_02x05_Odd_Even; footprint Connector_JST:JST_PH_B6B-PH-K_1x06_P2.00mm_Vertical -> Connector_PinHeader_2.54mm:PinHeader_2x05_P2.54mm_Vertical
- Q2, Q3, Q7: value NPN -> BC856B
- Q5, Q6: value NPN -> BC846
- R1: value 1k -> 0
- R11, R13, R18, R22, R23: value 1k -> 10k
- R21, R24: value 560 -> 10k
- R25: value 1k -> 100
- R26: value 10k -> 100
- R5: value 100k -> 100
- R6: value 10k -> 100k
- U1: value ESP32-WROOM-32D -> LD1117S33TR_SOT223; footprint ESP32-WROOM-32D:MODULE_ESP32-WROOM-32D -> Package_TO_SOT_SMD:SOT-223-3_TabPin2
- U2: value LD1117S33TR_SOT223 -> ESP32-WROOM-32D; footprint Package_TO_SOT_SMD:SOT-223-3_TabPin2 -> RF_Module:ESP32-WROOM-32
- moved J5 93.0 mm to (96.5, 3.00)
- moved J4 89.8 mm to (3.50, 13.0), turned to 90 degrees
- moved R12 74.0 mm to (91.5, 9.00), turned to 0 degrees
- moved R2 73.3 mm to (76.5, 14.0), turned to 0 degrees
- moved R5 72.0 mm to (3.00, 22.5)
- moved C1 70.9 mm to (80.5, 6.00), turned to 270 degrees
- moved R17 65.1 mm to (17.5, 10.0), turned to 180 degrees
- moved D3 64.8 mm to (72.0, 14.0), turned to 180 degrees
- moved R13 59.1 mm to (91.5, 5.00), turned to 0 degrees
- moved R26 58.3 mm to (8.50, 5.00), turned to 180 degrees
- moved C2 53.9 mm to (67.5, 5.85), turned to 90 degrees
- moved R15 53.0 mm to (29.5, 4.00), turned to 90 degrees
- moved R25 49.2 mm to (91.5, 11.0), turned to 0 degrees
- moved R22 48.0 mm to (8.50, 7.00), turned to 180 degrees
- moved R19 46.4 mm to (64.0, 12.0), turned to 180 degrees
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Connections:
- C1 pad 1: +5V -> +5VD
- J3 pad 2: Net-(J3-Pad2) -> TX0
- J3 pad 3: Net-(J3-Pad3) -> RX0
- J4 pad 1: Net-(J4-Pad1) -> GND
- J4 pad 2: VP -> 2VR
- J4 pad 3: GPIO33 -> 2ZF
- J4 pad 4: VN -> 2M
- J4 pad 5: GPIO32 -> 2EL
- J4 pad 6: GPIO35 -> +5VD
- J5 pad 1: Net-(J5-Pad1) -> GND
- J5 pad 2: 2EL -> 1VR
- J5 pad 3: 2M -> 1ZF
- J5 pad 4: 2ZF -> 1M
- J5 pad 5: 2VR -> 1EL
- J5 pad 6: GND -> +5VD
- J6 pad 1: Net-(J6-Pad1) -> GND
- J6 pad 2: 1EL -> VP
- J6 pad 3: 1M -> GPIO33
- J6 pad 4: 1ZF -> VN
- J6 pad 5: 1VR -> GPIO32
- J6 pad 6: GND -> GPIO35
- Q2 pad 2: GPIO4 -> +5VD
- Q2 pad 3: 1ZF -> 1VR
- Q3 pad 2: 1M -> +3V3
- Q4 pad 2: GPIO5 -> GPIO4
- Q4 pad 3: 2ZF -> 1ZF
- Q5 pad 2: 2M -> GND
- Q5 pad 3: GPIO23 -> Net-(Q5-Pad3)
- Q6 pad 2: GPIO18 -> GND
- Q6 pad 3: 1VR -> Net-(Q6-Pad3)
- Q7 pad 2: GPIO19 -> +5VD
- R10 pad 1: +3V3 -> +5VD
- R10 pad 2: GPIO22 -> 1ZF
- R11 pad 1: TX0 -> Net-(Q5-Pad1)
- R11 pad 2: Net-(J3-Pad2) -> GPIO18
- R12 pad 1: +5V -> Net-(Q6-Pad1)
- R12 pad 2: 2ZF -> 1M
- R13 pad 1: RX0 -> GND
- R13 pad 2: Net-(J3-Pad3) -> 1VR
- R14 pad 1: Net-(Q5-Pad1) -> GND
- R14 pad 2: +3V3 -> GPIO22
- R15 pad 1: Net-(Q6-Pad1) -> Net-(Q9-Pad1)
- R16 pad 1: +3V3 -> Net-(Q7-Pad1)
- R16 pad 2: GPIO23 -> Net-(Q10-Pad3)
- R17 pad 1: +5V -> Net-(Q8-Pad1)
- R17 pad 2: 1VR -> Net-(Q11-Pad3)
- R18 pad 1: GPIO18 -> +3V3
- R18 pad 2: GND -> EN
- R19 pad 1: Net-(Q7-Pad1) -> +3V3
- R19 pad 2: +3V3 -> GPIO0
- R20 pad 1: +5V -> +5VD
- R20 pad 2: 2VR -> 2ZF
- R21 pad 1: Net-(R21-Pad1) -> Net-(Q10-Pad1)
- R21 pad 2: 1EL -> GPIO19
- R22 pad 1: Net-(R21-Pad1) -> Net-(Q11-Pad1)
- R22 pad 2: GND -> 2M
- R23 pad 1: GPIO19 -> GND
- R23 pad 2: GND -> 2VR
- R24 pad 1: Net-(R24-Pad1) -> GND
- R24 pad 2: 2EL -> GPIO23
- R25 pad 1: Net-(R24-Pad1) -> GPIO25
- R25 pad 2: GND -> 1EL
- R26 pad 1: GPIO25 -> GPIO26
- R26 pad 2: +3V3 -> 2EL
- R5 pad 1: GND -> Net-(R5-Pad1)
- R5 pad 2: Net-(D4-Pad2) -> GPIO16
- R6 pad 1: Net-(Q2-Pad1) -> GND
- R6 pad 2: +3V3 -> Net-(D4-Pad2)
- R7 pad 1: +5V -> Net-(Q4-Pad1)
- R7 pad 2: 1ZF -> +3V3
- R8 pad 1: Net-(Q3-Pad1) -> Net-(Q2-Pad1)
- R8 pad 2: +3V3 -> Net-(Q5-Pad3)
- R9 pad 1: Net-(Q4-Pad1) -> Net-(Q3-Pad1)
- R9 pad 2: +3V3 -> Net-(Q6-Pad3)
- U1 pad 3: EN -> +5VD
- U2 pad 3: +5V -> EN
Routing:
- net +5VD: track 0.00 -> 127.6 mm, vias 0 -> 3
- net +5V: track 121.6 -> 16.5 mm, vias 6 -> 0
- net +3V3: track 176.8 -> 126.5 mm, vias 4 -> 9
- net EN: track 55.0 -> 6.09 mm, vias 1 -> 0
- net 1ZF: track 14.3 -> 61.0 mm, vias 0 -> 2
- net 1VR: track 13.5 -> 59.5 mm, vias 0 -> 1
- net GPIO18: track 59.0 -> 14.9 mm, vias 2 -> 0
- net 2EL: track 47.3 -> 4.09 mm, vias 1 -> 0
- net 1EL: track 45.8 -> 4.09 mm, vias 1 -> 0
- net GND: track 302.3 -> 337.2 mm, vias 30 -> 28
- net Net-(Q6-Pad1): track 4.11 -> 36.8 mm
- net GPIO22: track 58.6 -> 28.0 mm
- net TX0: track 29.5 -> 6.01 mm, vias 2 -> 0
- net GPIO4: track 43.8 -> 20.4 mm
- net GPIO19: track 42.1 -> 18.7 mm
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Other:
- outline, holes or cut-outs redrawn
- board text added: "+"
- board text added: "-"
- board text added: "1EL"
- board text added: "1M"
- board text added: "1VR"
- board text added: "1ZF"
- board text added: "2EL"
- board text added: "2M"
- board text added: "2VR"
- board text added: "2ZF"
- board text added: "Driver v2"
