File: driver_v0.2/driver.sch (KiCad schematic (older format))
At the start: 52 parts, among them J1 Pwr, J2 Batt, J3 isp, J5 Conn_01x06, J6 Conn_01x06, K1 Brake, Q1 IRF540N, Q2 NPN, Q3 NPN, Q4 NPN, Q5 NPN, Q6 NPN, Q7 NPN, U1 ESP32-WROOM-32D, U2 LD1117S33TR_SOT223, U3 MCP6044T-I_ST

Commit message: 2021-09-04
Parts:
- removed J3: isp, Connector_JST:JST_PH_B6B-PH-K_1x06_P2.00mm_Vertical, symbol Connector_Generic:Conn_01x06
- removed K1: Brake, OPL_Switch:SW4-6.0X6.0X5.0MM, symbol driver-rescue:DIP-SWITCH-TACTILE-SPST-NO_TS-1109_4P-D6.0MM_-OPL_Switch
- removed Q3, Q7: NPN, Package_TO_SOT_SMD:SOT-23, symbol Device:Q_NPN_BEC
- removed R10, R15, R20, R27: 10k, Resistor_SMD:R_0603_1608Metric_Pad0.98x0.95mm_HandSolder, symbol Device:R
- removed U3: MCP6044T-I_ST, MCP6044T:MCP6044T, symbol MCP6044T-I_ST:MCP6044T-I_ST
- added J3: Conn_01x04, Connector_PinHeader_2.54mm:PinHeader_1x04_P2.54mm_Vertical, symbol Connector_Generic:Conn_01x04
- added Q10, Q11: BC846, Package_TO_SOT_SMD:SOT-23, symbol Device:Q_NPN_BEC
- added Q2, Q3, Q7, Q8: BC856B, Package_TO_SOT_SMD:SOT-23, symbol Device:Q_PNP_BEC
- added R12, R9: 10k, Resistor_SMD:R_0603_1608Metric_Pad0.98x0.95mm_HandSolder, symbol Device:R
- added R5: 100, Resistor_SMD:R_0603_1608Metric_Pad0.98x0.95mm_HandSolder, symbol Device:R
- added SW1: SW_Push, Button_Switch_THT:SW_PUSH_6mm, symbol Switch:SW_Push
- Q1: value IRF540N -> F540N; Field4 (none) -> F540N
- Q5, Q6: value NPN -> BC846; MPN S8050 -> (none)
- R1: value 1k -> 0
- R11, R13, R18, R22, R23: value 1k -> 10k
- R21, R24: value 560 -> 10k
- R25: value 1k -> 100
- R26: value 10k -> 100
- U2: renamed from U1; footprint ESP32-WROOM-32D:MODULE_ESP32-WROOM-32D -> RF_Module:ESP32-WROOM-32
- gave numbers to parts that had none: 1
- renumbered J5 to J4, J6 to J5, Q2 to Q4, Q4 to Q9, R7 to R10, R9 to R15, R12 to R20, R5 to R6, R6 to R7, U2 to U1
Connections:
- net +3V3: now also R18.1, R19.1, J3.1 (Pin_1), Q3.2 (E), Q8.2 (E); no longer R14.2, R16.1, R19.2, R26.2, R8.2
- net +5V: no longer C1.1, R10.1, R17.1, R20.1, U1.3 (VI)
- net 1EL: now also J5.5 (Pin_5), R25.2; no longer J5.2 (Pin_2), R21.2
- net 1M: now also J5.4 (Pin_4), R12.2; no longer J5.3 (Pin_3)
- net 1VR: now also J5.2 (Pin_2), R13.2, Q2.3 (C); no longer J5.5 (Pin_5), Q6.3 (C), R17.2
- net 1ZF: now also J5.3 (Pin_3); no longer J5.4 (Pin_4)
- net 2EL: now also J4.5 (Pin_5), R26.2; no longer J4.2 (Pin_2), R24.2
- net 2M: now also J4.4 (Pin_4), R22.2; no longer J4.3 (Pin_3), Q5.2 (E)
- net 2VR: now also J4.2 (Pin_2), R23.2, Q7.3 (C); no longer J4.5 (Pin_5)
- net 2ZF: now also J4.3 (Pin_3); no longer J4.4 (Pin_4)
- net EN: now also R18.2
- net GND: now also J4.1 (Pin_1), J5.1 (Pin_1), J6.1 (Pin_1), Q5.2 (E), Q6.2 (E), R13.1, R14.1, R23.1, R24.1, J3.4 (Pin_4), Q10.2 (E), Q11.2 (E), SW1.1; no longer J4.6 (Pin_6), J5.6 (Pin_6), R18.2, R22.2, R23.2, R25.2
- net GPIO0: now also R19.2
- net GPIO16: now also R5.2
- net GPIO18: now also R11.2; no longer Q6.2 (E), R18.1
- net GPIO19: now also R21.2; no longer R23.1
- net GPIO22: now also R14.2, Q3.3 (C)
- net GPIO23: now also R24.2, Q8.3 (C); no longer Q5.3 (C), R16.2
- net GPIO25: now also R25.1; no longer R26.1
- net GPIO26: now also R26.1
- net RX0: now also J3.3 (Pin_3); no longer R13.1
- net TX0: now also J3.2 (Pin_2); no longer R11.1
- net at R21.1: now also Q10.1 (B); no longer R22.1
- net at Q6.1 (B): now also R12.1
- net at R8.1: now also Q2.1 (B)
- net at Q5.1 (B): now also R11.1; no longer R14.1
- new net: Q5.3 (C), R8.2
- new net: Q10.3 (C), R16.2
- new net: Q7.1 (B), R16.1
- new net: Q11.1 (B), R22.1
- new net: Q11.3 (C), R17.2
- new net: Q8.1 (B), R17.1
- new net: Q6.3 (C), R9.2
- new net: Q3.1 (B), R9.1
- new net: R5.1, SW1.2
- new net +5VD: C1.1, J4.6 (Pin_6), J5.6 (Pin_6), Q2.2 (E), Q7.2 (E), R10.1, R20.1, U1.3 (VI)
Other:
- moved on the sheet: C1, C2, C3, D3, J1, J6, Q4, Q9, R10, R15, R2, R20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
