File: controller_v0.2/controller.kicad_pcb (KiCad board)
At the start: 2 copper layers, 55 x 77.5 mm, 50 parts, among them J1 Battery, J2 USB_B_Micro, J3 isp, SW1 Power On/Off, SW2 Pairing, SW3 brake, U1 MCP73831-2-OT, U2 MIC5318-3.3YD5-TR, U3 ESP32-WROOM-32D, U4 Joystick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

Commit message: 2021-11-08
Parts:
- removed C10: 0.1u, Capacitor_SMD:C_0603_1608Metric_Pad1.08x0.95mm_HandSolder
- removed R16, R17: 1k, Resistor_SMD:R_0603_1608Metric_Pad0.98x0.95mm_HandSolder
- removed REF** (x4), e: MountingHole_3.2mm_M3, MountingHole:MountingHole_3.2mm_M3
- removed U5: MAX17048G+T10, MAX17048G_T10:MAX17048G_T10
- added D8: zenor/3.3v, Diode_THT:D_T-1_P5.08mm_Horizontal, F.Cu at (48.0, 28.0)
- added Q1: S8050, Package_TO_SOT_SMD:SOT-23, F.Cu at (48.0, 17.5)
- R14: value 10k -> 100
- R15: value 10k -> 1k
- moved R14 39.1 mm to (44.0, 16.5)
- moved R15 37.5 mm to (44.0, 18.5)
- moved R12 13.0 mm to (8.50, 15.0), turned to 0 degrees
- moved R11 8.50 mm to (8.50, 17.0), turned to 0 degrees
- moved R9 1.50 mm to (27.5, 49.5)
Connections:
- net GPIO15 renamed Net-(U3-Pad23)
- net Net-(C3-Pad1) renamed V_BATT
- D2 pad 2: GPIO2 -> GPIO4
- D6 pad 2: GPIO12 -> GPIO13
- J3 pad 2: Net-(J3-Pad2) -> TX0
- J3 pad 3: Net-(J3-Pad3) -> RX0
- R11 pad 1: TX0 -> EN
- R12 pad 1: GPIO5 -> GPIO0
- R14 pad 1: GPIO18 -> Net-(Q1-Pad1)
- R14 pad 2: +3V3 -> GPIO5
- R15 pad 1: GPIO19 -> Net-(Q1-Pad2)
- R15 pad 2: +3V3 -> GPIO33
- U3 pad 14: GPIO12 -> Net-(U3-Pad14)
- U3 pad 24: GPIO2 -> Net-(U3-Pad24)
Routing:
- net GPIO4: track 0.00 -> 45.9 mm, vias 0 -> 3
- net GPIO2: track 41.7 -> 0.00 mm, vias 3 -> 0
- net GPIO19: track 29.0 -> 0.00 mm, vias 1 -> 0
- net GPIO18: track 27.3 -> 0.00 mm, vias 1 -> 0
- net GPIO13: track 0.00 -> 22.2 mm, vias 0 -> 1
- net Net-(C6-Pad1): track 58.8 -> 36.8 mm
- net Earth: track 399.9 -> 378.9 mm, vias 19 -> 15
- net GPIO12: track 19.1 -> 0.00 mm, vias 1 -> 0
- net GPIO33: track 0.00 -> 14.7 mm, vias 0 -> 1
- net +3V3: track 110.5 -> 120.2 mm
- net +BATT: track 65.2 -> 56.1 mm
- net V_BATT: track 40.4 -> 49.2 mm
- net EN: track 40.1 -> 47.5 mm, vias 4 -> 3
- net RX0: track 15.5 -> 21.3 mm
- net Net-(J3-Pad3): track 5.09 -> 0.00 mm
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