File: controller_v0.2/controller.sch (KiCad schematic (older format))
At the start: 45 parts, among them J1 Battery, J2 USB_B_Micro, J3 isp, SW1 Power On/Off, SW2 Pairing, SW3 brake, U1 MCP73831-2-OT, U2 MIC5318-3.3YD5-TR, U3 ESP32-WROOM-32D, U4 Joystick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

Commit message: 2021-09-04
Parts:
- SW2, SW3: symbol OPL_Switch:DIP-SWITCH-TACTILE-SPST-NO_TS-1109_4P-D6.0MM_ -> controller-rescue:DIP-SWITCH-TACTILE-SPST-NO_TS-1109_4P-D6.0MM_-OPL_Switch
Changed lines of the file:
@@
 Sheet 1 1
 Title "Controller"
-Date "2021-07-05"
-Rev "v0.2"
+Date "2021-08-19"
+Rev "v1.0"
 Comp "Rotom"
 Comment1 ""
@@
 $EndComp
 $Comp
-L OPL_Switch:DIP-SWITCH-TACTILE-SPST-NO_TS-1109_4P-D6.0MM_ SW2
+L controller-rescue:DIP-SWITCH-TACTILE-SPST-NO_TS-1109_4P-D6.0MM_-OPL_Switch SW2
 U 1 1 60D03FEC
 P 5350 3750
@@
 	5450 4400 5250 4400
 $Comp
-L OPL_Switch:DIP-SWITCH-TACTILE-SPST-NO_TS-1109_4P-D6.0MM_ SW3
+L controller-rescue:DIP-SWITCH-TACTILE-SPST-NO_TS-1109_4P-D6.0MM_-OPL_Switch SW3
 U 1 1 60D12F78
 P 6100 3750

Commit message: 2021-11-08
Parts:
- removed C10: 0.1u, Capacitor_SMD:C_0603_1608Metric_Pad1.08x0.95mm_HandSolder, symbol Device:C
- removed R16, R17: 1k, Resistor_SMD:R_0603_1608Metric_Pad0.98x0.95mm_HandSolder, symbol Device:R
- removed U5: MAX17048G+T10, MAX17048G_T10:MAX17048G_T10, symbol MAX17048G_T10:MAX17048G+T10
- added D8: zenor/3.3v, Diode_THT:D_T-1_P5.08mm_Horizontal, symbol Diode:ZMMxx
- added Q1: S8050, Package_TO_SOT_SMD:SOT-23, symbol Device:Q_NPN_BEC
- R14: value 10k -> 100; MPN AC0603JR-0710KL -> (none)
- R15: value 10k -> 1k; MPN AC0603JR-0710KL -> (none)
Connections:
- net +3V3: no longer R14.2, R15.2
- net EN: now also R11.1
- net Earth: now also Q1.3 (C)
- net GPIO0: now also R12.1
- net GPIO13: now also D6.2 (A)
- net GPIO18: no longer R14.1
- net GPIO19: no longer R15.1
- net GPIO33: now also R15.2, D8.2 (A)
- net GPIO4: now also D2.2 (A)
- net GPIO5: now also R14.2; no longer R12.1
- net RX0: now also J3.3 (Pin_3)
- net TX0: now also J3.2 (Pin_2); no longer R11.1
- net V_BATT: now reaches C3.1, SW1.2 (B), U2.1 (IN), U2.3 (EN)
- net V_BATT: now also D8.1 (K)
- net GPIO12: no longer names the net of U3.14 (IO12)
- net GPIO12: no longer D6.2 (A)
- net GPIO15: no longer names the net of U3.23 (IO15)
- net GPIO2: no longer names the net of U3.24 (IO2)
- net GPIO2: no longer D2.2 (A)
- new net: Q1.2 (E), R15.1
- new net: Q1.1 (B), R14.1
- no-connect marks 0 -> 3
Other:
- moved on the sheet: R11, R12
