File: driver_v0.3/battery_level.sch (KiCad schematic (older format))
At the start: 18 parts

Commit message: 2021-11-08
Parts:
- gave numbers to parts that had none: 18
Connections:
- net Earth renamed BATT_GND
Changed lines of the file:
@@
 $EndDescr
 $Comp
-L Diode:1N53xxB D?
+L Diode:1N53xxB D2
 U 1 1 61332002
 P 3800 2050
-F 0 "D?" H 3800 2267 50  0000 C CNN
+F 0 "D2" H 3800 2267 50  0000 C CNN
 F 1 "zenor/32v" H 3800 2176 50  0000 C CNN
 F 2 "Diode_SMD:D_SOD-123" H 3800 1875 50  0001 C CNN
@@
 $EndComp
 $Comp
-L Diode:1N53xxB D?
+L Diode:1N53xxB D3
 U 1 1 613320F6
 P 4400 2050
-F 0 "D?" H 4400 2267 50  0000 C CNN
+F 0 "D3" H 4400 2267 50  0000 C CNN
 F 1 "zenor/2v" H 4400 2176 50  0000 C CNN
 F 2 "Diode_SMD:D_SOD-523" H 4400 1875 50  0001 C CNN
@@
 $EndComp
 $Comp
-L Diode:1N53xxB D?
+L Diode:1N53xxB D8
 U 1 1 61332980
 P 3650 2600
-F 0 "D?" H 3600 2400 50  0000 L CNN
+F 0 "D8" H 3600 2400 50  0000 L CNN
 F 1 "zenor/3.3v" H 3550 2500 50  0000 L CNN
 F 2 "Diode_SMD:D_SOD-323" H 3650 2425 50  0001 C CNN
@@
 $EndComp
 $Comp
-L Diode:1N53xxB D?
+L Diode:1N53xxB D4
 U 1 1 61334227
 P 4900 2050
-F 0 "D?" H 4900 2267 50  0000 C CNN
+F 0 "D4" H 4900 2267 50  0000 C CNN
 F 1 "zenor/2v" H 4900 2176 50  0000 C CNN
 F 2 "Diode_SMD:D_SOD-523" H 4900 1875 50  0001 C CNN
@@
 $EndComp
 $Comp
-L Diode:1N53xxB D?
+L Diode:1N53xxB D5
 U 1 1 61334A8C
 P 5400 2050
-F 0 "D?" H 5400 2267 50  0000 C CNN
+F 0 "D5" H 5400 2267 50  0000 C CNN
 F 1 "zenor/2v" H 5400 2176 50  0000 C CNN
 F 2 "Diode_SMD:D_SOD-523" H 5400 1875 50  0001 C CNN
@@
 $EndComp
 $Comp
-L Diode:1N53xxB D?
+L Diode:1N53xxB D6
 U 1 1 61335545
 P 5900 2050
-F 0 "D?" H 5900 2267 50  0000 C CNN
+F 0 "D6" H 5900 2267 50  0000 C CNN
 F 1 "zenor/2v" H 5900 2176 50  0000 C CNN
 F 2 "Diode_SMD:D_SOD-523" H 5900 1875 50  0001 C CNN
@@
 $EndComp
 $Comp
-L Diode:1N53xxB D?
+L Diode:1N53xxB D7
 U 1 1 613356C6
 P 6400 2050
-F 0 "D?" H 6400 2267 50  0000 C CNN
+F 0 "D7" H 6400 2267 50  0000 C CNN
 F 1 "zenor/2v" H 6400 2176 50  0000 C CNN
 F 2 "Diode_SMD:D_SOD-523" H 6400 1875 50  0001 C CNN
@@
 	1    0    0    -1
 $EndComp
-$Comp
-L power:Earth #PWR?
-U 1 1 61335905
-P 6550 2050
-F 0 "#PWR?" H 6550 1800 50  0001 C CNN
-F 1 "Earth" H 6550 1900 50  0001 C CNN
-F 2 "" H 6550 2050 50  0001 C CNN
-F 3 "~" H 6550 2050 50  0001 C CNN
-	1    6550 2050
-	0    -1   -1   0
-$EndComp
 Wire Wire Line
 	6250 2050 6150 2050
@@
 	4150 2050 4050 2050
 $Comp
-L Device:R R?
+L Device:R R8
 U 1 1 6133673B
 P 4150 2300
-F 0 "R?" H 4080 2254 50  0000 R CNN
+F 0 "R8" H 4080 2254 50  0000 R CNN
 F 1 "560" H 4080 2345 50  0000 R CNN
 F 2 "Resistor_SMD:R_0603_1608Metric" V 4080 2300 50  0001 C CNN
@@
 $EndComp
 $Comp
-L Device:LED D?
+L Device:LED D9
 U 1 1 61336CA1
 P 4150 2600
-F 0 "D?" V 4189 2482 50  0000 R CNN
+F 0 "D9" V 4189 2482 50  0000 R CNN
 F 1 "RED" V 4098 2482 50  0000 R CNN
 F 2 "LED_SMD:LED_0805_2012Metric" H 4150 2600 50  0001 C CNN
@@
 Wire Wire Line
 	4750 2050 4650 2050
-$Comp
-L power:Earth #PWR?
-U 1 1 6133A02F
-P 4150 2750
-F 0 "#PWR?" H 4150 2500 50  0001 C CNN
-F 1 "Earth" H 4150 2600 50  0001 C CNN
-F 2 "" H 4150 2750 50  0001 C CNN
-F 3 "~" H 4150 2750 50  0001 C CNN
-	1    4150 2750
-	1    0    0    -1
-$EndComp
 Wire Wire Line
 	4650 2150 4650 2050
 $Comp
-L Device:R R?
+L Device:R R9
 U 1 1 6133AF22
 P 4650 2300
-F 0 "R?" H 4580 2254 50  0000 R CNN
+F 0 "R9" H 4580 2254 50  0000 R CNN
 F 1 "430" H 4580 2345 50  0000 R CNN
 F 2 "Resistor_SMD:R_0603_1608Metric" V 4580 2300 50  0001 C CNN
@@
 $EndComp
 $Comp
-L Device:LED D?
+L Device:LED D10
 U 1 1 6133AF29
 P 4650 2600
-F 0 "D?" V 4689 2482 50  0000 R CNN
+F 0 "D10" V 4689 2482 50  0000 R CNN
 F 1 "RED" V 4598 2482 50  0000 R CNN
 F 2 "LED_SMD:LED_0805_2012Metric" H 4650 2600 50  0001 C CNN
@@
 	0    -1   -1   0
 $EndComp
-$Comp
-L power:Earth #PWR?
-U 1 1 6133AF2F
-P 4650 2750
-F 0 "#PWR?" H 4650 2500 50  0001 C CNN
-F 1 "Earth" H 4650 2600 50  0001 C CNN
-F 2 "" H 4650 2750 50  0001 C CNN
-F 3 "~" H 4650 2750 50  0001 C CNN
-	1    4650 2750
-	1    0    0    -1
-$EndComp
 Wire Wire Line
 	5150 2150 5150 2050
 $Comp
-L Device:R R?
+L Device:R R10
 U 1 1 6133B09F
 P 5150 2300
-F 0 "R?" H 5080 2254 50  0000 R CNN
+F 0 "R10" H 5080 2254 50  0000 R CNN
 F 1 "280" H 5080 2345 50  0000 R CNN
 F 2 "Resistor_SMD:R_0603_1608Metric" V 5080 2300 50  0001 C CNN
@@
 $EndComp
 $Comp
-L Device:LED D?
+L Device:LED D11
 U 1 1 6133B0A6
 P 5150 2600
-F 0 "D?" V 5189 2482 50  0000 R CNN
+F 0 "D11" V 5189 2482 50  0000 R CNN
 F 1 "RED" V 5098 2482 50  0000 R CNN
 F 2 "LED_SMD:LED_0805_2012Metric" H 5150 2600 50  0001 C CNN
@@
 	0    -1   -1   0
 $EndComp
-$Comp
-L power:Earth #PWR?
-U 1 1 6133B0AC
-P 5150 2750
-F 0 "#PWR?" H 5150 2500 50  0001 C CNN
-F 1 "Earth" H 5150 2600 50  0001 C CNN
-F 2 "" H 5150 2750 50  0001 C CNN
-F 3 "~" H 5150 2750 50  0001 C CNN
-	1    5150 2750
-	1    0    0    -1
-$EndComp
 Wire Wire Line
 	5650 2150 5650 2050
 $Comp
-L Device:R R?
+L Device:R R11
 U 1 1 6133B1CC
 P 5650 2300
-F 0 "R?" H 5580 2254 50  0000 R CNN
+F 0 "R11" H 5580 2254 50  0000 R CNN
 F 1 "150" H 5580 2345 50  0000 R CNN
 F 2 "Resistor_SMD:R_0603_1608Metric" V 5580 2300 50  0001 C CNN
@@
 $EndComp
 $Comp
-L Device:LED D?
+L Device:LED D12
 U 1 1 6133B1D3
 P 5650 2600
-F 0 "D?" V 5689 2482 50  0000 R CNN
+F 0 "D12" V 5689 2482 50  0000 R CNN
 F 1 "RED" V 5598 2482 50  0000 R CNN
 F 2 "LED_SMD:LED_0805_2012Metric" H 5650 2600 50  0001 C CNN
@@
 	0    -1   -1   0
 $EndComp
-$Comp
-L power:Earth #PWR?
-U 1 1 6133B1D9
-P 5650 2750
-F 0 "#PWR?" H 5650 2500 50  0001 C CNN
-F 1 "Earth" H 5650 2600 50  0001 C CNN
-F 2 "" H 5650 2750 50  0001 C CNN
-F 3 "~" H 5650 2750 50  0001 C CNN
-	1    5650 2750
-	1    0    0    -1
-$EndComp
 Wire Wire Line
 	6150 2150 6150 2050
 $Comp
-L Device:R R?
+L Device:R R12
 U 1 1 6133B302
 P 6150 2300
-F 0 "R?" H 6080 2254 50  0000 R CNN
+F 0 "R12" H 6080 2254 50  0000 R CNN
 F 1 "100" H 6080 2345 50  0000 R CNN
 F 2 "Resistor_SMD:R_0603_1608Metric" V 6080 2300 50  0001 C CNN
@@
 $EndComp
 $Comp
-L Device:LED D?
+L Device:LED D13
 U 1 1 6133B309
 P 6150 2600
-F 0 "D?" V 6189 2482 50  0000 R CNN
+F 0 "D13" V 6189 2482 50  0000 R CNN
 F 1 "RED" V 6098 2482 50  0000 R CNN
 F 2 "LED_SMD:LED_0805_2012Metric" H 6150 2600 50  0001 C CNN
@@
 	0    -1   -1   0
 $EndComp
-$Comp
-L power:Earth #PWR?
-U 1 1 6133B30F
-P 6150 2750
-F 0 "#PWR?" H 6150 2500 50  0001 C CNN
-F 1 "Earth" H 6150 2600 50  0001 C CNN
-F 2 "" H 6150 2750 50  0001 C CNN
-F 3 "~" H 6150 2750 50  0001 C CNN
-	1    6150 2750
-	1    0    0    -1
-$EndComp
 Connection ~ 4650 2050
 Wire Wire Line
@@
 	6150 2050 6050 2050
 $Comp
-L Device:R R?
+L Device:R R7
 U 1 1 6133BA16
 P 3650 2300
-F 0 "R?" H 3580 2254 50  0000 R CNN
+F 0 "R7" H 3580 2254 50  0000 R CNN
 F 1 "100k" H 3580 2345 50  0000 R CNN
 F 2 "Resistor_SMD:R_0603_1608Metric" V 3580 2300 50  0001 C CNN
@@
 	-1   0    0    1
 $EndComp
-$Comp
-L power:Earth #PWR?
-U 1 1 6133C7F8
-P 3650 2750
-F 0 "#PWR?" H 3650 2500 50  0001 C CNN
-F 1 "Earth" H 3650 2600 50  0001 C CNN
-F 2 "" H 3650 2750 50  0001 C CNN
-F 3 "~" H 3650 2750 50  0001 C CNN
-	1    3650 2750
-	1    0    0    -1
-$EndComp
 Wire Wire Line
 	3450 2450 3650 2450
@@
 	3950 2050 4050 2050
 Connection ~ 4050 2050
+Text HLabel 3450 3000 0    50   Input ~ 0
+BATT_GND
+Wire Wire Line
+	3650 2750 3650 3000
+Wire Wire Line
+	3650 3000 3450 3000
+Wire Wire Line
+	3650 2750 4150 2750
+Connection ~ 3650 2750
+Connection ~ 4150 2750
+Wire Wire Line
+	4150 2750 4650 2750
+Connection ~ 4650 2750
+Wire Wire Line
+	4650 2750 5150 2750
+Connection ~ 5150 2750
+Wire Wire Line
+	5150 2750 5650 2750
+Connection ~ 5650 2750
+Wire Wire Line
+	5650 2750 6150 2750
+Wire Wire Line
+	6550 2050 6550 2750
+Wire Wire Line
+	6550 2750 6150 2750
+Connection ~ 6150 2750
 $EndSCHEMATC
