File: driver_v0.3/driver_v0.3.sch (KiCad schematic (older format))
At the start: 19 parts

Commit message: 2021-11-08
Parts:
- added J1, J2: Conn_01x03, Connector_PinHeader_2.54mm:PinHeader_1x03_P2.54mm_Vertical, symbol Connector_Generic:Conn_01x03
- D1: renamed from D?; footprint (none) -> LED_SMD:LED_0805_2012Metric_Pad1.15x1.40mm_HandSolder
- gave numbers to parts that had none: 18
Connections:
- net Earth: now also J1.1 (Pin_1)
- net IO34(LVSENS): now also J1.3 (Pin_3)
- net V_BATT: now also J1.2 (Pin_2)
- new net Battery Level Guage/BATT_10CELL: J2.2 (Pin_2)
- new net Battery Level Guage/BATT_GND: J2.1 (Pin_1)
- new net Battery Level Guage/BATT_SENS: J2.3 (Pin_3)
